File: Electronics/02_Board_files/01_Project files/V1_Flight_Controller/V1_Flight_Controller.brd (EAGLE design)
At the start: 46.2 x 46.2 mm, 27 parts, among them J101 JTAG_CONNECTOR, U101 STM32F030K6T6, U201 MPU-6050, Y1 8MHz

Commit message: 1. Created hierarchical structure in schematic 2. Battery charging and protection circuit added 3. Added various eagle libraries
Parts:
- removed C101, C102, C103, C104, C105, C106, C107: (no value), adafruit:C0603
- removed C201: 0.1uF, 4V, ±10%, adafruit:C0603
- removed C202: 10nF, 4V, ±10%, adafruit:C0603
- removed C203: 2.2nF, 50V, ±10%, adafruit:C0603
- removed C204: 0.1uF, 2V, ±10%, adafruit:C0603
- removed J101: JTAG_CONNECTOR, con-molex:53047-05
- removed L101, L102, L103, L104, L201: (no value), rcl:L2012C
- removed R101: (no value), adafruit:R0603
- removed R201, R202: 4.7k, adafruit:R0603
- removed TP1, TP2, TP3: TPB1,27, testpad:B1,27
- removed U101: STM32F030K6T6, STM32F030K6T6:QFP80P900X900X160-32N
- removed U201: MPU-6050, MPU-6050:QFN50P400X400X95-24N
- removed U301: (no value), esp12e:ESP8266-ESP12E
- removed Y1: 8MHz, SparkFun-Clocks:HC49UP
- added BATTERY_PROTECTION_AND_MONITORING1:C1: 0.1uF, adafruit:C0603K
- added BATTERY_PROTECTION_AND_MONITORING1:C2: 10uF, adafruit:C0603K
- added BATTERY_PROTECTION_AND_MONITORING1:D101: GREEN_LED, adafruit:CHIPLED_0603
- added BATTERY_PROTECTION_AND_MONITORING1:D102: RED_LED, adafruit:CHIPLED_0603
- added BATTERY_PROTECTION_AND_MONITORING1:R1: 1.2KΩ, adafruit:R0603
- added BATTERY_PROTECTION_AND_MONITORING1:R2, BATTERY_PROTECTION_AND_MONITORING1:R3, BATTERY_PROTECTION_AND_MONITORING1:R4: 1KΩ, adafruit:R0603
- added BATTERY_PROTECTION_AND_MONITORING1:R5: 100Ω, adafruit:R0603
- added BATTERY_PROTECTION_AND_MONITORING1:T1: DMN3024LSD, FS8205A:TSSOP-8
- added BATTERY_PROTECTION_AND_MONITORING1:TP1, MICROCONTROLLER1:TP1, MICROCONTROLLER1:TP2, MICROCONTROLLER1:TP3: TPB1,27, testpad:B1,27
- added BATTERY_PROTECTION_AND_MONITORING1:U101: TP4056, tp4056:SOP-8
- added BATTERY_PROTECTION_AND_MONITORING1:U102: DW01A, dw01a:SOT23-6
- added BATTERY_PROTECTION_AND_MONITORING1:U104: MICRO-USB, con-molex-usb:47589-0001
- added MICROCONTROLLER1:C101, MICROCONTROLLER1:C102: 100nF, adafruit:C0603
- added MICROCONTROLLER1:C103: 4.7uF, adafruit:C0603
- added MICROCONTROLLER1:C104: 10nF, adafruit:C0603
- added MICROCONTROLLER1:C105: 1uF, adafruit:C0603
- added MICROCONTROLLER1:C106, MICROCONTROLLER1:C107: 20pF, adafruit:C0603
- added MICROCONTROLLER1:L101, MICROCONTROLLER1:L102, MICROCONTROLLER1:L103, MICROCONTROLLER1:L104, SENSOR1:L201: (no value), rcl:L2012C
- added MICROCONTROLLER1:R101: 10KΩ, adafruit:R0603
- added MICROCONTROLLER1:U101: STM32F030K6T6, STM32F030K6T6:QFP80P900X900X160-32N
- added MICROCONTROLLER1:Y1: 8MHz, SparkFun-Clocks:HC49UP
- added SENSOR1:C201: 0.1uF, 4V, ±10%, adafruit:C0603
- added SENSOR1:C202: 10nF, 4V, ±10%, adafruit:C0603
- added SENSOR1:C203: 2.2nF, 50V, ±10%, adafruit:C0603
- added SENSOR1:C204: 0.1uF, 2V, ±10%, adafruit:C0603
- added SENSOR1:R201, SENSOR1:R202: 4.7k, adafruit:R0603
- added SENSOR1:U201: MPU-6050, MPU-6050:QFN50P400X400X95-24N
- added WIFI1:U301: (no value), esp12e:ESP8266-ESP12E
Connections:
- removed net 3V3: L101.2, L201.2, U301.8
- removed net 3V3_IMU: C201.1, C202.1, L201.1, R201.1, R202.1, U201.13, U201.8
- removed net 3V3_MCU: C101.1, C102.1, C103.1, J101.1, L101.1, L102.2, L104.1, R101.1, TP1.TP, U101.1, U101.17
- removed net BOOT0: L102.1, L103.1, U101.31
- removed net GND_IMU: C201.2, C202.2, C203.2, C204.2, U201.1, U201.11, U201.18, U201.9
- removed net GND_MCU: C101.2, C102.2, C103.2, C104.2, C105.2, C106.2, C107.2, J101.3, L103.2, U101.16, U101.32
- removed net I2C1_SCL: TP2.TP, U101.29
- removed net I2C1_SDA: TP3.TP, U101.30
- removed net IMU_INT: U201.12
- removed net N$1: C204.1, U201.10
- removed net N$2: C203.1, U201.20
- removed net NRST: J101.5, R101.2, U101.4
- removed net PWM_PIN1: U101.18
- removed net PWM_PIN2: U101.19
- removed net PWM_PIN3: U101.20
- removed net PWM_PIN4: U101.21
- removed net RST: U301.1
- removed net SCL: R201.2, U201.23
- removed net SDA: R202.2, U201.24
- removed net SWCLK: J101.2, U101.24
- removed net SWDIO: J101.4, U101.23
- removed net USART1_RX: U101.9
- removed net USART1_TX: U101.8
- removed net VBAT_LEVEL: U101.6
- removed net VDDA: C104.1, C105.1, L104.2, U101.5
- removed net XTAL_IN: C106.1, U101.2, Y1.1
- removed net XTAL_OUT: C107.1, U101.3, Y1.2
- new net +3V3: MICROCONTROLLER1:L101.2, SENSOR1:L201.2
- new net BATTERY_+VE: BATTERY_PROTECTION_AND_MONITORING1:C2.1, BATTERY_PROTECTION_AND_MONITORING1:R5.2, BATTERY_PROTECTION_AND_MONITORING1:U101.5
- new net BATTERY_-VE: BATTERY_PROTECTION_AND_MONITORING1:C1.2, BATTERY_PROTECTION_AND_MONITORING1:T1.2, BATTERY_PROTECTION_AND_MONITORING1:T1.3, BATTERY_PROTECTION_AND_MONITORING1:U102.6
- new net BATTERY_PROTECTION_AND_MONITORING1:+5V: BATTERY_PROTECTION_AND_MONITORING1:D101.A, BATTERY_PROTECTION_AND_MONITORING1:D102.A, BATTERY_PROTECTION_AND_MONITORING1:U101.4, BATTERY_PROTECTION_AND_MONITORING1:U101.8, BATTERY_PROTECTION_AND_MONITORING1:U104.1
- new net BATTERY_PROTECTION_AND_MONITORING1:N$1: BATTERY_PROTECTION_AND_MONITORING1:R1.2, BATTERY_PROTECTION_AND_MONITORING1:U101.2
- new net BATTERY_PROTECTION_AND_MONITORING1:N$2: BATTERY_PROTECTION_AND_MONITORING1:R4.1, BATTERY_PROTECTION_AND_MONITORING1:U101.6
- new net BATTERY_PROTECTION_AND_MONITORING1:N$3: BATTERY_PROTECTION_AND_MONITORING1:R2.1, BATTERY_PROTECTION_AND_MONITORING1:U101.7
- new net BATTERY_PROTECTION_AND_MONITORING1:N$4: BATTERY_PROTECTION_AND_MONITORING1:D101.C, BATTERY_PROTECTION_AND_MONITORING1:D102.C, BATTERY_PROTECTION_AND_MONITORING1:R2.2, BATTERY_PROTECTION_AND_MONITORING1:R4.2
- new net BATTERY_PROTECTION_AND_MONITORING1:N$5: BATTERY_PROTECTION_AND_MONITORING1:TP1.TP, BATTERY_PROTECTION_AND_MONITORING1:U102.4
- new net BATTERY_PROTECTION_AND_MONITORING1:N$6: BATTERY_PROTECTION_AND_MONITORING1:T1.1, BATTERY_PROTECTION_AND_MONITORING1:T1.8
- new net BATTERY_PROTECTION_AND_MONITORING1:N$7: BATTERY_PROTECTION_AND_MONITORING1:R3.2, BATTERY_PROTECTION_AND_MONITORING1:U102.2
- new net BATTERY_PROTECTION_AND_MONITORING1:N$8: BATTERY_PROTECTION_AND_MONITORING1:C1.1, BATTERY_PROTECTION_AND_MONITORING1:R5.1, BATTERY_PROTECTION_AND_MONITORING1:U102.5
- new net BATTERY_PROTECTION_AND_MONITORING1:OC: BATTERY_PROTECTION_AND_MONITORING1:T1.5, BATTERY_PROTECTION_AND_MONITORING1:U102.3
- new net BATTERY_PROTECTION_AND_MONITORING1:OD: BATTERY_PROTECTION_AND_MONITORING1:T1.4, BATTERY_PROTECTION_AND_MONITORING1:U102.1
- new net ESP8266_RST: MICROCONTROLLER1:U101.7, WIFI1:U301.1
- new net MICROCONTROLLER1:3V3_MCU: MICROCONTROLLER1:C101.1, MICROCONTROLLER1:C102.1, MICROCONTROLLER1:C103.1, MICROCONTROLLER1:L101.1, MICROCONTROLLER1:L102.2, MICROCONTROLLER1:L104.1, MICROCONTROLLER1:R101.1, MICROCONTROLLER1:TP1.TP, MICROCONTROLLER1:U101.1, MICROCONTROLLER1:U101.17
- new net MICROCONTROLLER1:BOOT0: MICROCONTROLLER1:L102.1, MICROCONTROLLER1:L103.1, MICROCONTROLLER1:U101.31
- new net MICROCONTROLLER1:GND_MCU: MICROCONTROLLER1:C101.2, MICROCONTROLLER1:C102.2, MICROCONTROLLER1:C103.2, MICROCONTROLLER1:C104.2, MICROCONTROLLER1:C105.2, MICROCONTROLLER1:C106.2, MICROCONTROLLER1:C107.2, MICROCONTROLLER1:L103.2, MICROCONTROLLER1:U101.16, MICROCONTROLLER1:U101.32
- new net MICROCONTROLLER1:I2C1_SCL: MICROCONTROLLER1:TP2.TP, MICROCONTROLLER1:U101.29
- new net MICROCONTROLLER1:I2C1_SDA: MICROCONTROLLER1:TP3.TP, MICROCONTROLLER1:U101.30
- new net MICROCONTROLLER1:NRST: MICROCONTROLLER1:R101.2, MICROCONTROLLER1:U101.4
- new net MICROCONTROLLER1:PWM_PIN1: MICROCONTROLLER1:U101.18
- new net MICROCONTROLLER1:PWM_PIN2: MICROCONTROLLER1:U101.19
- new net MICROCONTROLLER1:PWM_PIN3: MICROCONTROLLER1:U101.20
- new net MICROCONTROLLER1:PWM_PIN4: MICROCONTROLLER1:U101.21
- new net MICROCONTROLLER1:SWCLK: MICROCONTROLLER1:U101.24
- new net MICROCONTROLLER1:SWDIO: MICROCONTROLLER1:U101.23
- new net MICROCONTROLLER1:VBAT_LEVEL: MICROCONTROLLER1:U101.6
- new net MICROCONTROLLER1:VDDA: MICROCONTROLLER1:C104.1, MICROCONTROLLER1:C105.1, MICROCONTROLLER1:L104.2, MICROCONTROLLER1:U101.5
- new net MICROCONTROLLER1:XTAL_IN: MICROCONTROLLER1:C106.1, MICROCONTROLLER1:U101.2, MICROCONTROLLER1:Y1.1
- new net MICROCONTROLLER1:XTAL_OUT: MICROCONTROLLER1:C107.1, MICROCONTROLLER1:U101.3, MICROCONTROLLER1:Y1.2
- new net SENSOR1:3V3_IMU: SENSOR1:C201.1, SENSOR1:C202.1, SENSOR1:L201.1, SENSOR1:R201.1, SENSOR1:R202.1, SENSOR1:U201.13, SENSOR1:U201.8
- new net SENSOR1:GND_IMU: SENSOR1:C201.2, SENSOR1:C202.2, SENSOR1:C203.2, SENSOR1:C204.2, SENSOR1:U201.1, SENSOR1:U201.11, SENSOR1:U201.18, SENSOR1:U201.9
- new net SENSOR1:IMU_INT: SENSOR1:U201.12
- new net SENSOR1:N$1: SENSOR1:C204.1, SENSOR1:U201.10
- new net SENSOR1:N$2: SENSOR1:C203.1, SENSOR1:U201.20
- new net SENSOR1:SCL: SENSOR1:R201.2, SENSOR1:U201.23
- new net SENSOR1:SDA: SENSOR1:R202.2, SENSOR1:U201.24
- new net UART1_RX: MICROCONTROLLER1:U101.9, WIFI1:U301.16
- new net UART1_TX: MICROCONTROLLER1:U101.8, WIFI1:U301.15
- new net WIFI1:3V3_ESP8266: WIFI1:U301.8
- new net WIFI1:GND_ESP8266: WIFI1:U301.9
- net GND: now also BATTERY_PROTECTION_AND_MONITORING1:C2.2, BATTERY_PROTECTION_AND_MONITORING1:R1.1, BATTERY_PROTECTION_AND_MONITORING1:R3.1, BATTERY_PROTECTION_AND_MONITORING1:T1.6, BATTERY_PROTECTION_AND_MONITORING1:T1.7, BATTERY_PROTECTION_AND_MONITORING1:U101.1, BATTERY_PROTECTION_AND_MONITORING1:U101.3, BATTERY_PROTECTION_AND_MONITORING1:U104.5, BATTERY_PROTECTION_AND_MONITORING1:U104.CASING1, BATTERY_PROTECTION_AND_MONITORING1:U104.CASING2, BATTERY_PROTECTION_AND_MONITORING1:U104.CASING3, BATTERY_PROTECTION_AND_MONITORING1:U104.CASING4; no longer U301.9

Commit message: 1. added connectors 2. added imu_int 3. added block diagram linkages 4. overall clean up
Parts:
- removed BATTERY_PROTECTION_AND_MONITORING1:U104: MICRO-USB, con-molex-usb:47589-0001
- added CONNECTORS1:U104: MICRO-USB, con-molex-usb:47589-0001
- added CONNECTORS1:X1: Battery Connector, con-jst:SM02B-SRSS-TB
- added CONNECTORS1:X2: Motor 1, con-jst:SM02B-SRSS-TB
- added CONNECTORS1:X3: Motor 2, con-jst:SM02B-SRSS-TB
- added CONNECTORS1:X4: Motor 3, con-jst:SM02B-SRSS-TB
- added CONNECTORS1:X5: Motor 4, con-jst:SM02B-SRSS-TB
- added CONNECTORS1:X6: JTAG, con-molex:53047-05
- added MICROCONTROLLER1:R102: 2KΩ, adafruit:R0603
- added MICROCONTROLLER1:R2: 5KΩ, adafruit:R0603
Connections:
- net MICROCONTROLLER1:I2C1_SCL renamed I2C_SCL
- net MICROCONTROLLER1:I2C1_SDA renamed I2C_SDA
- removed net BATTERY_PROTECTION_AND_MONITORING1:+5V: BATTERY_PROTECTION_AND_MONITORING1:D101.A, BATTERY_PROTECTION_AND_MONITORING1:D102.A, BATTERY_PROTECTION_AND_MONITORING1:U101.4, BATTERY_PROTECTION_AND_MONITORING1:U101.8, BATTERY_PROTECTION_AND_MONITORING1:U104.1
- removed net MICROCONTROLLER1:NRST: MICROCONTROLLER1:R101.2, MICROCONTROLLER1:U101.4
- removed net MICROCONTROLLER1:SWCLK: MICROCONTROLLER1:U101.24
- removed net MICROCONTROLLER1:SWDIO: MICROCONTROLLER1:U101.23
- new net +5V: BATTERY_PROTECTION_AND_MONITORING1:D101.A, BATTERY_PROTECTION_AND_MONITORING1:D102.A, BATTERY_PROTECTION_AND_MONITORING1:U101.4, BATTERY_PROTECTION_AND_MONITORING1:U101.8, CONNECTORS1:U104.1
- new net MICROCONTROLLER1:BAT_MON: MICROCONTROLLER1:R102.1, MICROCONTROLLER1:R2.2, MICROCONTROLLER1:U101.6
- new net MICROCONTROLLER1:IMU_INT: MICROCONTROLLER1:U101.10
- new net N$10: CONNECTORS1:X4.2
- new net N$11: CONNECTORS1:X2.2
- new net N$12: CONNECTORS1:X3.2
- new net N$13: CONNECTORS1:X5.2
- new net NRST: CONNECTORS1:X6.5, MICROCONTROLLER1:R101.2, MICROCONTROLLER1:U101.4
- new net SWCLK: CONNECTORS1:X6.2, MICROCONTROLLER1:U101.24
- new net SWDIO: CONNECTORS1:X6.4, MICROCONTROLLER1:U101.23
- net +3V3: now also CONNECTORS1:X6.1
- net BATTERY_+VE: now also CONNECTORS1:X1.1, CONNECTORS1:X2.1, CONNECTORS1:X3.1, CONNECTORS1:X4.1, CONNECTORS1:X5.1
- net BATTERY_-VE: now also CONNECTORS1:X1.2
- net GND: now also CONNECTORS1:U104.5, CONNECTORS1:U104.CASING1, CONNECTORS1:U104.CASING2, CONNECTORS1:U104.CASING3, CONNECTORS1:U104.CASING4, CONNECTORS1:X6.3; no longer BATTERY_PROTECTION_AND_MONITORING1:U104.5, BATTERY_PROTECTION_AND_MONITORING1:U104.CASING1, BATTERY_PROTECTION_AND_MONITORING1:U104.CASING2, BATTERY_PROTECTION_AND_MONITORING1:U104.CASING3, BATTERY_PROTECTION_AND_MONITORING1:U104.CASING4
- net MICROCONTROLLER1:GND_MCU: now also MICROCONTROLLER1:R2.1
- net MICROCONTROLLER1:VBAT_LEVEL: now also MICROCONTROLLER1:R102.2; no longer MICROCONTROLLER1:U101.6

Commit message: 1. Completed schematic 2. Added/Created required libraries/footprints
Parts:
- added 3V3_BUCK_CONVERTER1:C1, 3V3_BUCK_CONVERTER1:C2: (no value), adafruit:C0603K
- added 3V3_BUCK_CONVERTER1:D201: GREEN_LED, adafruit:CHIPLED_0603
- added 3V3_BUCK_CONVERTER1:R1, MOTOR_CONTROL1:R1, MOTOR_CONTROL1:R2, MOTOR_CONTROL1:R3, MOTOR_CONTROL1:R4, MOTOR_CONTROL1:R5, MOTOR_CONTROL1:R6, MOTOR_CONTROL1:R7, MOTOR_CONTROL1:R8: (no value), adafruit:R0603
- added 3V3_BUCK_CONVERTER1:U$1: LM3670, smd-footprints:SOT-23-5
- added 3V3_BUCK_CONVERTER1:U$2: SRN2009T-2R2M, SRN2009T-2R2M:SRN2009T-2R2M
- added MOTOR_CONTROL1:Q1, MOTOR_CONTROL1:Q2, MOTOR_CONTROL1:Q3, MOTOR_CONTROL1:Q4: (no value), adafruit:SOT23
- added MOTOR_CONTROL1:U$1, MOTOR_CONTROL1:U$2, MOTOR_CONTROL1:U$3, MOTOR_CONTROL1:U$4: SS310-SCHOTTKY, SS310-SCHOTTKY:SS310-SCHOTTKY
Connections:
- removed net MICROCONTROLLER1:PWM_PIN1: MICROCONTROLLER1:U101.18
- removed net MICROCONTROLLER1:PWM_PIN2: MICROCONTROLLER1:U101.19
- removed net MICROCONTROLLER1:PWM_PIN3: MICROCONTROLLER1:U101.20
- removed net MICROCONTROLLER1:PWM_PIN4: MICROCONTROLLER1:U101.21
- removed net N$10: CONNECTORS1:X4.2
- removed net N$11: CONNECTORS1:X2.2
- removed net N$12: CONNECTORS1:X3.2
- removed net N$13: CONNECTORS1:X5.2
- new net 3V3_BUCK_CONVERTER1:N$1: 3V3_BUCK_CONVERTER1:U$1.5, 3V3_BUCK_CONVERTER1:U$2.1
- new net 3V3_BUCK_CONVERTER1:N$2: 3V3_BUCK_CONVERTER1:D201.A, 3V3_BUCK_CONVERTER1:R1.1
- new net M1: CONNECTORS1:X2.2, MOTOR_CONTROL1:Q1.3, MOTOR_CONTROL1:U$1.P$1
- new net M1_PWM: MICROCONTROLLER1:U101.18, MOTOR_CONTROL1:R1.1
- new net M2: CONNECTORS1:X3.2, MOTOR_CONTROL1:Q2.3, MOTOR_CONTROL1:U$2.P$1
- new net M2_PWM: MICROCONTROLLER1:U101.19, MOTOR_CONTROL1:R3.1
- new net M3: CONNECTORS1:X4.2, MOTOR_CONTROL1:Q3.3, MOTOR_CONTROL1:U$3.P$1
- new net M3_PWM: MICROCONTROLLER1:U101.20, MOTOR_CONTROL1:R5.1
- new net M4: CONNECTORS1:X5.2, MOTOR_CONTROL1:Q4.3, MOTOR_CONTROL1:U$4.P$1
- new net M4_PWM: MICROCONTROLLER1:U101.21, MOTOR_CONTROL1:R7.1
- new net MOTOR_CONTROL1:N$1: MOTOR_CONTROL1:Q2.1, MOTOR_CONTROL1:R3.2, MOTOR_CONTROL1:R4.2
- new net MOTOR_CONTROL1:N$2: MOTOR_CONTROL1:Q1.1, MOTOR_CONTROL1:R1.2, MOTOR_CONTROL1:R2.2
- new net MOTOR_CONTROL1:N$3: MOTOR_CONTROL1:Q3.1, MOTOR_CONTROL1:R5.2, MOTOR_CONTROL1:R6.2
- new net MOTOR_CONTROL1:N$4: MOTOR_CONTROL1:Q4.1, MOTOR_CONTROL1:R7.2, MOTOR_CONTROL1:R8.2
- net +3V3: now also 3V3_BUCK_CONVERTER1:C2.1, 3V3_BUCK_CONVERTER1:R1.2, 3V3_BUCK_CONVERTER1:U$1.4, 3V3_BUCK_CONVERTER1:U$2.2
- net BATTERY_+VE: now also 3V3_BUCK_CONVERTER1:C1.1, 3V3_BUCK_CONVERTER1:U$1.1, 3V3_BUCK_CONVERTER1:U$1.3, MOTOR_CONTROL1:U$1.P$2, MOTOR_CONTROL1:U$2.P$2, MOTOR_CONTROL1:U$3.P$2, MOTOR_CONTROL1:U$4.P$2
- net GND: now also 3V3_BUCK_CONVERTER1:C1.2, 3V3_BUCK_CONVERTER1:C2.2, 3V3_BUCK_CONVERTER1:D201.C, 3V3_BUCK_CONVERTER1:U$1.2, MOTOR_CONTROL1:Q1.2, MOTOR_CONTROL1:Q2.2, MOTOR_CONTROL1:Q3.2, MOTOR_CONTROL1:Q4.2, MOTOR_CONTROL1:R2.1, MOTOR_CONTROL1:R4.1, MOTOR_CONTROL1:R6.1, MOTOR_CONTROL1:R8.1

Commit message: 1. Made changes in a few libraries, and added new footprints/libraries 2. Placement progress - 80%
Parts:
- removed 3V3_BUCK_CONVERTER1:C1, 3V3_BUCK_CONVERTER1:C2: (no value), adafruit:C0603K
- removed 3V3_BUCK_CONVERTER1:D201, BATTERY_PROTECTION_AND_MONITORING1:D101: GREEN_LED, adafruit:CHIPLED_0603
- removed 3V3_BUCK_CONVERTER1:R1, MOTOR_CONTROL1:R1, MOTOR_CONTROL1:R2, MOTOR_CONTROL1:R3, MOTOR_CONTROL1:R4, MOTOR_CONTROL1:R5, MOTOR_CONTROL1:R6, MOTOR_CONTROL1:R7, MOTOR_CONTROL1:R8: (no value), adafruit:R0603
- removed 3V3_BUCK_CONVERTER1:U$1: LM3670, smd-footprints:SOT-23-5
- removed 3V3_BUCK_CONVERTER1:U$2: SRN2009T-2R2M, SRN2009T-2R2M:SRN2009T-2R2M
- removed BATTERY_PROTECTION_AND_MONITORING1:C1: 0.1uF, adafruit:C0603K
- removed BATTERY_PROTECTION_AND_MONITORING1:C2: 10uF, adafruit:C0603K
- removed BATTERY_PROTECTION_AND_MONITORING1:D102: RED_LED, adafruit:CHIPLED_0603
- removed BATTERY_PROTECTION_AND_MONITORING1:R1: 1.2KΩ, adafruit:R0603
- removed BATTERY_PROTECTION_AND_MONITORING1:R2, BATTERY_PROTECTION_AND_MONITORING1:R3, BATTERY_PROTECTION_AND_MONITORING1:R4: 1KΩ, adafruit:R0603
- removed BATTERY_PROTECTION_AND_MONITORING1:R5: 100Ω, adafruit:R0603
- removed BATTERY_PROTECTION_AND_MONITORING1:T1: DMN3024LSD, FS8205A:TSSOP-8
- removed BATTERY_PROTECTION_AND_MONITORING1:TP1, MICROCONTROLLER1:TP1, MICROCONTROLLER1:TP2, MICROCONTROLLER1:TP3: TPB1,27, testpad:B1,27
- removed BATTERY_PROTECTION_AND_MONITORING1:U101: TP4056, tp4056:SOP-8
- removed BATTERY_PROTECTION_AND_MONITORING1:U102: DW01A, dw01a:SOT23-6
- removed CONNECTORS1:U104: MICRO-USB, con-molex-usb:47589-0001
- removed CONNECTORS1:X1: Battery Connector, con-jst:SM02B-SRSS-TB
- removed CONNECTORS1:X6: JTAG, con-molex:53047-05
- removed MICROCONTROLLER1:C101, MICROCONTROLLER1:C102: 100nF, adafruit:C0603
- removed MICROCONTROLLER1:C103: 4.7uF, adafruit:C0603
- removed MICROCONTROLLER1:C104: 10nF, adafruit:C0603
- removed MICROCONTROLLER1:C105: 1uF, adafruit:C0603
- removed MICROCONTROLLER1:C106, MICROCONTROLLER1:C107: 20pF, adafruit:C0603
- removed MICROCONTROLLER1:L101, MICROCONTROLLER1:L102, MICROCONTROLLER1:L103, MICROCONTROLLER1:L104, SENSOR1:L201: (no value), rcl:L2012C
- removed MICROCONTROLLER1:R101: 10KΩ, adafruit:R0603
- removed MICROCONTROLLER1:R102: 2KΩ, adafruit:R0603
- removed MICROCONTROLLER1:R2: 5KΩ, adafruit:R0603
- removed MICROCONTROLLER1:U101: STM32F030K6T6, STM32F030K6T6:QFP80P900X900X160-32N
- removed MICROCONTROLLER1:Y1: 8MHz, SparkFun-Clocks:HC49UP
- removed MOTOR_CONTROL1:Q1, MOTOR_CONTROL1:Q2, MOTOR_CONTROL1:Q3, MOTOR_CONTROL1:Q4: (no value), adafruit:SOT23
- removed MOTOR_CONTROL1:U$1, MOTOR_CONTROL1:U$2, MOTOR_CONTROL1:U$3, MOTOR_CONTROL1:U$4: SS310-SCHOTTKY, SS310-SCHOTTKY:SS310-SCHOTTKY
- removed SENSOR1:C201: 0.1uF, 4V, ±10%, adafruit:C0603
- removed SENSOR1:C202: 10nF, 4V, ±10%, adafruit:C0603
- removed SENSOR1:C203: 2.2nF, 50V, ±10%, adafruit:C0603
- removed SENSOR1:C204: 0.1uF, 2V, ±10%, adafruit:C0603
- removed SENSOR1:R201, SENSOR1:R202: 4.7k, adafruit:R0603
- removed SENSOR1:U201: MPU-6050, MPU-6050:QFN50P400X400X95-24N
- removed WIFI1:U301: (no value), esp12e:ESP8266-ESP12E
- added 01_BATTERY_PROTECTION_AND_MONITORING:C1: 0.1uF, adafruit:C0603K
- added 01_BATTERY_PROTECTION_AND_MONITORING:C2: 10uF, adafruit:C0603K
- added 01_BATTERY_PROTECTION_AND_MONITORING:D101, 02_3V3_BUCK_CONVERTER:D201: GREEN_LED, adafruit:CHIPLED_0603
- added 01_BATTERY_PROTECTION_AND_MONITORING:D102: RED_LED, adafruit:CHIPLED_0603
- added 01_BATTERY_PROTECTION_AND_MONITORING:R101: 1.2KΩ, adafruit:R0603
- added 01_BATTERY_PROTECTION_AND_MONITORING:R102, 01_BATTERY_PROTECTION_AND_MONITORING:R103, 01_BATTERY_PROTECTION_AND_MONITORING:R105: 1KΩ, adafruit:R0603
- added 01_BATTERY_PROTECTION_AND_MONITORING:R104: 100Ω, adafruit:R0603
- added 01_BATTERY_PROTECTION_AND_MONITORING:T101: DMN3024LSD, FS8205A:TSSOP-8
- added 01_BATTERY_PROTECTION_AND_MONITORING:TP_5V, 01_BATTERY_PROTECTION_AND_MONITORING:TP_B+, 01_BATTERY_PROTECTION_AND_MONITORING:TP_TD, 02_3V3_BUCK_CONVERTER:TP_3V3, 02_3V3_BUCK_CONVERTER:TP_BUCK_VIN, 03_MICROCONTROLLER:TP_MCU_3V3, 03_MICROCONTROLLER:TP_SCL, 03_MICROCONTROLLER:TP_SDA, 05_SENSOR:TP_IMU_3V3, 06_MOTOR_CONTROL:TP_M1, 06_MOTOR_CONTROL:TP_M2, 06_MOTOR_CONTROL:TP_M3, 06_MOTOR_CONTROL:TP_M4, 07_CONNECTORS:TP_B+, 07_CONNECTORS:TP_B-: TPB1,27, testpad:B1,27
- added 01_BATTERY_PROTECTION_AND_MONITORING:U101: TP4056, tp4056:SOP-8
- added 01_BATTERY_PROTECTION_AND_MONITORING:U102: DW01A, dw01a:SOT23-6
- added 02_3V3_BUCK_CONVERTER:C201, 02_3V3_BUCK_CONVERTER:C202: (no value), adafruit:C0603K
- added 02_3V3_BUCK_CONVERTER:L201: SRN2009T-2R2M, SRN2009T-2R2M:SRN2009T-2R2M
- added 02_3V3_BUCK_CONVERTER:R201, 06_MOTOR_CONTROL:R601, 06_MOTOR_CONTROL:R602, 06_MOTOR_CONTROL:R603, 06_MOTOR_CONTROL:R604, 06_MOTOR_CONTROL:R605, 06_MOTOR_CONTROL:R606, 06_MOTOR_CONTROL:R607, 06_MOTOR_CONTROL:R608: (no value), adafruit:R0603
- added 02_3V3_BUCK_CONVERTER:U201: LM3670, smd-footprints:SOT-23-5
- added 03_MICROCONTROLLER:C301, 03_MICROCONTROLLER:C302: 100nF, adafruit:C0603
- added 03_MICROCONTROLLER:C303: 4.7uF, adafruit:C0603
- added 03_MICROCONTROLLER:C304: 10nF, adafruit:C0603
- added 03_MICROCONTROLLER:C305: 1uF, adafruit:C0603
- added 03_MICROCONTROLLER:C306, 03_MICROCONTROLLER:C307: 20pF, adafruit:C0603
- added 03_MICROCONTROLLER:L301, 03_MICROCONTROLLER:L302, 03_MICROCONTROLLER:L303, 03_MICROCONTROLLER:L304, 05_SENSOR:L501: (no value), rcl:L2012C
- added 03_MICROCONTROLLER:R301: 10KΩ, adafruit:R0603
- added 03_MICROCONTROLLER:R302: 2KΩ, adafruit:R0603
- added 03_MICROCONTROLLER:R303: 5KΩ, adafruit:R0603
- added 03_MICROCONTROLLER:U301: STM32F030K6T6, STM32F030K6T6:QFP80P900X900X160-32N
- added 03_MICROCONTROLLER:Y301: 8MHz, SparkFun-Clocks:HC49UP
- added 04_WIFI:U401: (no value), esp12e:ESP8266-ESP12E
- added 05_SENSOR:C501: 0.1uF, 4V, ±10%, adafruit:C0603
- added 05_SENSOR:C502: 10nF, 4V, ±10%, adafruit:C0603
- added 05_SENSOR:C503: 2.2nF, 50V, ±10%, adafruit:C0603
- added 05_SENSOR:C504: 0.1uF, 2V, ±10%, adafruit:C0603
- added 05_SENSOR:R501, 05_SENSOR:R502: 4.7k, adafruit:R0603
- added 05_SENSOR:U501: MPU-6050, MPU-6050:QFN50P400X400X95-24N
- added 06_MOTOR_CONTROL:D601, 06_MOTOR_CONTROL:D602, 06_MOTOR_CONTROL:D603, 06_MOTOR_CONTROL:D604: (no value), diode:SOD123
- added 06_MOTOR_CONTROL:Q601, 06_MOTOR_CONTROL:Q602, 06_MOTOR_CONTROL:Q603, 06_MOTOR_CONTROL:Q604: (no value), adafruit:SOT23
- added 07_CONNECTORS:J701: MICRO-USB, con-molex-usb:47589-0001
- added 07_CONNECTORS:X701: Battery Connector, con-jst:SM02B-SRSS-TB
- added 07_CONNECTORS:X706: JTAG, con-molex:53047-05
- renumbered CONNECTORS1:X2 to 07_CONNECTORS:X702, CONNECTORS1:X3 to 07_CONNECTORS:X703, CONNECTORS1:X4 to 07_CONNECTORS:X704, CONNECTORS1:X5 to 07_CONNECTORS:X705
Connections:
- removed net 3V3_BUCK_CONVERTER1:N$1: 3V3_BUCK_CONVERTER1:U$1.5, 3V3_BUCK_CONVERTER1:U$2.1
- removed net 3V3_BUCK_CONVERTER1:N$2: 3V3_BUCK_CONVERTER1:D201.A, 3V3_BUCK_CONVERTER1:R1.1
- removed net BATTERY_PROTECTION_AND_MONITORING1:N$1: BATTERY_PROTECTION_AND_MONITORING1:R1.2, BATTERY_PROTECTION_AND_MONITORING1:U101.2
- removed net BATTERY_PROTECTION_AND_MONITORING1:N$2: BATTERY_PROTECTION_AND_MONITORING1:R4.1, BATTERY_PROTECTION_AND_MONITORING1:U101.6
- removed net BATTERY_PROTECTION_AND_MONITORING1:N$3: BATTERY_PROTECTION_AND_MONITORING1:R2.1, BATTERY_PROTECTION_AND_MONITORING1:U101.7
- removed net BATTERY_PROTECTION_AND_MONITORING1:N$4: BATTERY_PROTECTION_AND_MONITORING1:D101.C, BATTERY_PROTECTION_AND_MONITORING1:D102.C, BATTERY_PROTECTION_AND_MONITORING1:R2.2, BATTERY_PROTECTION_AND_MONITORING1:R4.2
- removed net BATTERY_PROTECTION_AND_MONITORING1:N$5: BATTERY_PROTECTION_AND_MONITORING1:TP1.TP, BATTERY_PROTECTION_AND_MONITORING1:U102.4
- removed net BATTERY_PROTECTION_AND_MONITORING1:N$6: BATTERY_PROTECTION_AND_MONITORING1:T1.1, BATTERY_PROTECTION_AND_MONITORING1:T1.8
- removed net BATTERY_PROTECTION_AND_MONITORING1:N$7: BATTERY_PROTECTION_AND_MONITORING1:R3.2, BATTERY_PROTECTION_AND_MONITORING1:U102.2
- removed net BATTERY_PROTECTION_AND_MONITORING1:N$8: BATTERY_PROTECTION_AND_MONITORING1:C1.1, BATTERY_PROTECTION_AND_MONITORING1:R5.1, BATTERY_PROTECTION_AND_MONITORING1:U102.5
- removed net BATTERY_PROTECTION_AND_MONITORING1:OC: BATTERY_PROTECTION_AND_MONITORING1:T1.5, BATTERY_PROTECTION_AND_MONITORING1:U102.3
- removed net BATTERY_PROTECTION_AND_MONITORING1:OD: BATTERY_PROTECTION_AND_MONITORING1:T1.4, BATTERY_PROTECTION_AND_MONITORING1:U102.1
- removed net MICROCONTROLLER1:3V3_MCU: MICROCONTROLLER1:C101.1, MICROCONTROLLER1:C102.1, MICROCONTROLLER1:C103.1, MICROCONTROLLER1:L101.1, MICROCONTROLLER1:L102.2, MICROCONTROLLER1:L104.1, MICROCONTROLLER1:R101.1, MICROCONTROLLER1:TP1.TP, MICROCONTROLLER1:U101.1, MICROCONTROLLER1:U101.17
- removed net MICROCONTROLLER1:BAT_MON: MICROCONTROLLER1:R102.1, MICROCONTROLLER1:R2.2, MICROCONTROLLER1:U101.6
- removed net MICROCONTROLLER1:BOOT0: MICROCONTROLLER1:L102.1, MICROCONTROLLER1:L103.1, MICROCONTROLLER1:U101.31
- removed net MICROCONTROLLER1:GND_MCU: MICROCONTROLLER1:C101.2, MICROCONTROLLER1:C102.2, MICROCONTROLLER1:C103.2, MICROCONTROLLER1:C104.2, MICROCONTROLLER1:C105.2, MICROCONTROLLER1:C106.2, MICROCONTROLLER1:C107.2, MICROCONTROLLER1:L103.2, MICROCONTROLLER1:R2.1, MICROCONTROLLER1:U101.16, MICROCONTROLLER1:U101.32
- removed net MICROCONTROLLER1:IMU_INT: MICROCONTROLLER1:U101.10
- removed net MICROCONTROLLER1:VBAT_LEVEL: MICROCONTROLLER1:R102.2
- removed net MICROCONTROLLER1:VDDA: MICROCONTROLLER1:C104.1, MICROCONTROLLER1:C105.1, MICROCONTROLLER1:L104.2, MICROCONTROLLER1:U101.5
- removed net MICROCONTROLLER1:XTAL_IN: MICROCONTROLLER1:C106.1, MICROCONTROLLER1:U101.2, MICROCONTROLLER1:Y1.1
- removed net MICROCONTROLLER1:XTAL_OUT: MICROCONTROLLER1:C107.1, MICROCONTROLLER1:U101.3, MICROCONTROLLER1:Y1.2
- removed net MOTOR_CONTROL1:N$1: MOTOR_CONTROL1:Q2.1, MOTOR_CONTROL1:R3.2, MOTOR_CONTROL1:R4.2
- removed net MOTOR_CONTROL1:N$2: MOTOR_CONTROL1:Q1.1, MOTOR_CONTROL1:R1.2, MOTOR_CONTROL1:R2.2
- removed net MOTOR_CONTROL1:N$3: MOTOR_CONTROL1:Q3.1, MOTOR_CONTROL1:R5.2, MOTOR_CONTROL1:R6.2
- removed net MOTOR_CONTROL1:N$4: MOTOR_CONTROL1:Q4.1, MOTOR_CONTROL1:R7.2, MOTOR_CONTROL1:R8.2
- removed net SENSOR1:3V3_IMU: SENSOR1:C201.1, SENSOR1:C202.1, SENSOR1:L201.1, SENSOR1:R201.1, SENSOR1:R202.1, SENSOR1:U201.13, SENSOR1:U201.8
- removed net SENSOR1:GND_IMU: SENSOR1:C201.2, SENSOR1:C202.2, SENSOR1:C203.2, SENSOR1:C204.2, SENSOR1:U201.1, SENSOR1:U201.11, SENSOR1:U201.18, SENSOR1:U201.9
- removed net SENSOR1:IMU_INT: SENSOR1:U201.12
- removed net SENSOR1:N$1: SENSOR1:C204.1, SENSOR1:U201.10
- removed net SENSOR1:N$2: SENSOR1:C203.1, SENSOR1:U201.20
- removed net SENSOR1:SCL: SENSOR1:R201.2, SENSOR1:U201.23
- removed net SENSOR1:SDA: SENSOR1:R202.2, SENSOR1:U201.24
- removed net WIFI1:3V3_ESP8266: WIFI1:U301.8
- removed net WIFI1:GND_ESP8266: WIFI1:U301.9
- new net 01_BATTERY_PROTECTION_AND_MONITORING:CHRG: 01_BATTERY_PROTECTION_AND_MONITORING:R103.1, 01_BATTERY_PROTECTION_AND_MONITORING:U101.7
- new net 01_BATTERY_PROTECTION_AND_MONITORING:CHRG_LED: 01_BATTERY_PROTECTION_AND_MONITORING:D102.C, 01_BATTERY_PROTECTION_AND_MONITORING:R103.2
- new net 01_BATTERY_PROTECTION_AND_MONITORING:CS: 01_BATTERY_PROTECTION_AND_MONITORING:R105.2, 01_BATTERY_PROTECTION_AND_MONITORING:U102.2
- new net 01_BATTERY_PROTECTION_AND_MONITORING:N$6: 01_BATTERY_PROTECTION_AND_MONITORING:T101.1, 01_BATTERY_PROTECTION_AND_MONITORING:T101.8
- new net 01_BATTERY_PROTECTION_AND_MONITORING:OC: 01_BATTERY_PROTECTION_AND_MONITORING:T101.5, 01_BATTERY_PROTECTION_AND_MONITORING:U102.3
- new net 01_BATTERY_PROTECTION_AND_MONITORING:OD: 01_BATTERY_PROTECTION_AND_MONITORING:T101.4, 01_BATTERY_PROTECTION_AND_MONITORING:U102.1
- new net 01_BATTERY_PROTECTION_AND_MONITORING:PROG: 01_BATTERY_PROTECTION_AND_MONITORING:R101.2, 01_BATTERY_PROTECTION_AND_MONITORING:U101.2
- new net 01_BATTERY_PROTECTION_AND_MONITORING:STDBY: 01_BATTERY_PROTECTION_AND_MONITORING:R102.1, 01_BATTERY_PROTECTION_AND_MONITORING:U101.6
- new net 01_BATTERY_PROTECTION_AND_MONITORING:STDBY_LED: 01_BATTERY_PROTECTION_AND_MONITORING:D101.C, 01_BATTERY_PROTECTION_AND_MONITORING:R102.2
- new net 01_BATTERY_PROTECTION_AND_MONITORING:TD: 01_BATTERY_PROTECTION_AND_MONITORING:TP_TD.TP, 01_BATTERY_PROTECTION_AND_MONITORING:U102.4
- new net 01_BATTERY_PROTECTION_AND_MONITORING:VCC: 01_BATTERY_PROTECTION_AND_MONITORING:C1.1, 01_BATTERY_PROTECTION_AND_MONITORING:R104.1, 01_BATTERY_PROTECTION_AND_MONITORING:U102.5
- new net 02_3V3_BUCK_CONVERTER:N$1: 02_3V3_BUCK_CONVERTER:L201.1, 02_3V3_BUCK_CONVERTER:U201.5
- new net 02_3V3_BUCK_CONVERTER:N$2: 02_3V3_BUCK_CONVERTER:D201.A, 02_3V3_BUCK_CONVERTER:R201.1
- new net 03_MICROCONTROLLER:3V3_MCU: 03_MICROCONTROLLER:C301.1, 03_MICROCONTROLLER:C302.1, 03_MICROCONTROLLER:C303.1, 03_MICROCONTROLLER:L301.1, 03_MICROCONTROLLER:L302.2, 03_MICROCONTROLLER:L304.1, 03_MICROCONTROLLER:R301.1, 03_MICROCONTROLLER:TP_MCU_3V3.TP, 03_MICROCONTROLLER:U301.1, 03_MICROCONTROLLER:U301.17
- new net 03_MICROCONTROLLER:BAT_MON: 03_MICROCONTROLLER:R302.1, 03_MICROCONTROLLER:R303.2, 03_MICROCONTROLLER:U301.6
- new net 03_MICROCONTROLLER:BOOT0: 03_MICROCONTROLLER:L302.1, 03_MICROCONTROLLER:L303.1, 03_MICROCONTROLLER:U301.31
- new net 03_MICROCONTROLLER:GND_MCU: 03_MICROCONTROLLER:C301.2, 03_MICROCONTROLLER:C302.2, 03_MICROCONTROLLER:C303.2, 03_MICROCONTROLLER:C304.2, 03_MICROCONTROLLER:C305.2, 03_MICROCONTROLLER:C306.2, 03_MICROCONTROLLER:C307.2, 03_MICROCONTROLLER:L303.2, 03_MICROCONTROLLER:R303.1, 03_MICROCONTROLLER:U301.16, 03_MICROCONTROLLER:U301.32
- new net 03_MICROCONTROLLER:IMU_INT: 03_MICROCONTROLLER:U301.10
- new net 03_MICROCONTROLLER:VBAT_LEVEL: 03_MICROCONTROLLER:R302.2
- new net 03_MICROCONTROLLER:VDDA: 03_MICROCONTROLLER:C304.1, 03_MICROCONTROLLER:C305.1, 03_MICROCONTROLLER:L304.2, 03_MICROCONTROLLER:U301.5
- new net 03_MICROCONTROLLER:XTAL_IN: 03_MICROCONTROLLER:C306.1, 03_MICROCONTROLLER:U301.2, 03_MICROCONTROLLER:Y301.1
- new net 03_MICROCONTROLLER:XTAL_OUT: 03_MICROCONTROLLER:C307.1, 03_MICROCONTROLLER:U301.3, 03_MICROCONTROLLER:Y301.2
- new net 04_WIFI:3V3_ESP8266: 04_WIFI:U401.8
- new net 04_WIFI:GND_ESP8266: 04_WIFI:U401.9
- new net 05_SENSOR:3V3_IMU: 05_SENSOR:C501.1, 05_SENSOR:C502.1, 05_SENSOR:L501.1, 05_SENSOR:R501.1, 05_SENSOR:R502.1, 05_SENSOR:TP_IMU_3V3.TP, 05_SENSOR:U501.13, 05_SENSOR:U501.8
- new net 05_SENSOR:GND_IMU: 05_SENSOR:C501.2, 05_SENSOR:C502.2, 05_SENSOR:C503.2, 05_SENSOR:C504.2, 05_SENSOR:U501.1, 05_SENSOR:U501.11, 05_SENSOR:U501.18, 05_SENSOR:U501.9
- new net 05_SENSOR:IMU_INT: 05_SENSOR:U501.12
- new net 05_SENSOR:N$1: 05_SENSOR:C504.1, 05_SENSOR:U501.10
- new net 05_SENSOR:N$2: 05_SENSOR:C503.1, 05_SENSOR:U501.20
- new net 05_SENSOR:SCL: 05_SENSOR:R501.2, 05_SENSOR:U501.23
- new net 05_SENSOR:SDA: 05_SENSOR:R502.2, 05_SENSOR:U501.24
- new net 06_MOTOR_CONTROL:N$1: 06_MOTOR_CONTROL:Q602.1, 06_MOTOR_CONTROL:R603.2, 06_MOTOR_CONTROL:R604.2
- new net 06_MOTOR_CONTROL:N$2: 06_MOTOR_CONTROL:Q601.1, 06_MOTOR_CONTROL:R601.2, 06_MOTOR_CONTROL:R602.2
- new net 06_MOTOR_CONTROL:N$3: 06_MOTOR_CONTROL:Q603.1, 06_MOTOR_CONTROL:R605.2, 06_MOTOR_CONTROL:R606.2
- new net 06_MOTOR_CONTROL:N$4: 06_MOTOR_CONTROL:Q604.1, 06_MOTOR_CONTROL:R607.2, 06_MOTOR_CONTROL:R608.2
- net +3V3: now also 02_3V3_BUCK_CONVERTER:C202.1, 02_3V3_BUCK_CONVERTER:L201.2, 02_3V3_BUCK_CONVERTER:R201.2, 02_3V3_BUCK_CONVERTER:TP_3V3.TP, 02_3V3_BUCK_CONVERTER:U201.4, 03_MICROCONTROLLER:L301.2, 05_SENSOR:L501.2, 07_CONNECTORS:X706.1; no longer 3V3_BUCK_CONVERTER1:C2.1, 3V3_BUCK_CONVERTER1:R1.2, 3V3_BUCK_CONVERTER1:U$1.4, 3V3_BUCK_CONVERTER1:U$2.2, CONNECTORS1:X6.1, MICROCONTROLLER1:L101.2, SENSOR1:L201.2
- net +5V: now also 01_BATTERY_PROTECTION_AND_MONITORING:D101.A, 01_BATTERY_PROTECTION_AND_MONITORING:D102.A, 01_BATTERY_PROTECTION_AND_MONITORING:TP_5V.TP, 01_BATTERY_PROTECTION_AND_MONITORING:U101.4, 01_BATTERY_PROTECTION_AND_MONITORING:U101.8, 07_CONNECTORS:J701.1; no longer BATTERY_PROTECTION_AND_MONITORING1:D101.A, BATTERY_PROTECTION_AND_MONITORING1:D102.A, BATTERY_PROTECTION_AND_MONITORING1:U101.4, BATTERY_PROTECTION_AND_MONITORING1:U101.8, CONNECTORS1:U104.1
- net BATTERY_+VE: now also 01_BATTERY_PROTECTION_AND_MONITORING:C2.1, 01_BATTERY_PROTECTION_AND_MONITORING:R104.2, 01_BATTERY_PROTECTION_AND_MONITORING:TP_B+.TP, 01_BATTERY_PROTECTION_AND_MONITORING:U101.5, 02_3V3_BUCK_CONVERTER:C201.1, 02_3V3_BUCK_CONVERTER:TP_BUCK_VIN.TP, 02_3V3_BUCK_CONVERTER:U201.1, 02_3V3_BUCK_CONVERTER:U201.3, 06_MOTOR_CONTROL:D601.C, 06_MOTOR_CONTROL:D602.C, 06_MOTOR_CONTROL:D603.C, 06_MOTOR_CONTROL:D604.C, 06_MOTOR_CONTROL:TP_M1.TP, 06_MOTOR_CONTROL:TP_M2.TP, 06_MOTOR_CONTROL:TP_M3.TP, 06_MOTOR_CONTROL:TP_M4.TP, 07_CONNECTORS:TP_B+.TP, 07_CONNECTORS:X701.1; no longer 3V3_BUCK_CONVERTER1:C1.1, 3V3_BUCK_CONVERTER1:U$1.1, 3V3_BUCK_CONVERTER1:U$1.3, BATTERY_PROTECTION_AND_MONITORING1:C2.1, BATTERY_PROTECTION_AND_MONITORING1:R5.2, BATTERY_PROTECTION_AND_MONITORING1:U101.5, CONNECTORS1:X1.1, MOTOR_CONTROL1:U$1.P$2, MOTOR_CONTROL1:U$2.P$2, MOTOR_CONTROL1:U$3.P$2, MOTOR_CONTROL1:U$4.P$2
- net BATTERY_-VE: now also 01_BATTERY_PROTECTION_AND_MONITORING:C1.2, 01_BATTERY_PROTECTION_AND_MONITORING:T101.2, 01_BATTERY_PROTECTION_AND_MONITORING:T101.3, 01_BATTERY_PROTECTION_AND_MONITORING:U102.6, 07_CONNECTORS:TP_B-.TP, 07_CONNECTORS:X701.2; no longer BATTERY_PROTECTION_AND_MONITORING1:C1.2, BATTERY_PROTECTION_AND_MONITORING1:T1.2, BATTERY_PROTECTION_AND_MONITORING1:T1.3, BATTERY_PROTECTION_AND_MONITORING1:U102.6, CONNECTORS1:X1.2
- net ESP8266_RST: now also 03_MICROCONTROLLER:U301.7, 04_WIFI:U401.1; no longer MICROCONTROLLER1:U101.7, WIFI1:U301.1
- net GND: now also 01_BATTERY_PROTECTION_AND_MONITORING:C2.2, 01_BATTERY_PROTECTION_AND_MONITORING:R101.1, 01_BATTERY_PROTECTION_AND_MONITORING:R105.1, 01_BATTERY_PROTECTION_AND_MONITORING:T101.6, 01_BATTERY_PROTECTION_AND_MONITORING:T101.7, 01_BATTERY_PROTECTION_AND_MONITORING:U101.1, 01_BATTERY_PROTECTION_AND_MONITORING:U101.3, 02_3V3_BUCK_CONVERTER:C201.2, 02_3V3_BUCK_CONVERTER:C202.2, 02_3V3_BUCK_CONVERTER:D201.C, 02_3V3_BUCK_CONVERTER:U201.2, 06_MOTOR_CONTROL:Q601.2, 06_MOTOR_CONTROL:Q602.2, 06_MOTOR_CONTROL:Q603.2, 06_MOTOR_CONTROL:Q604.2, 06_MOTOR_CONTROL:R602.1, 06_MOTOR_CONTROL:R604.1, 06_MOTOR_CONTROL:R606.1, 06_MOTOR_CONTROL:R608.1, 07_CONNECTORS:J701.5, 07_CONNECTORS:J701.CASING1, 07_CONNECTORS:J701.CASING2, 07_CONNECTORS:J701.CASING3, 07_CONNECTORS:J701.CASING4, 07_CONNECTORS:X706.3; no longer 3V3_BUCK_CONVERTER1:C1.2, 3V3_BUCK_CONVERTER1:C2.2, 3V3_BUCK_CONVERTER1:D201.C, 3V3_BUCK_CONVERTER1:U$1.2, BATTERY_PROTECTION_AND_MONITORING1:C2.2, BATTERY_PROTECTION_AND_MONITORING1:R1.1, BATTERY_PROTECTION_AND_MONITORING1:R3.1, BATTERY_PROTECTION_AND_MONITORING1:T1.6, BATTERY_PROTECTION_AND_MONITORING1:T1.7, BATTERY_PROTECTION_AND_MONITORING1:U101.1, BATTERY_PROTECTION_AND_MONITORING1:U101.3, CONNECTORS1:U104.5, CONNECTORS1:U104.CASING1, CONNECTORS1:U104.CASING2, CONNECTORS1:U104.CASING3, CONNECTORS1:U104.CASING4, CONNECTORS1:X6.3, MOTOR_CONTROL1:Q1.2, MOTOR_CONTROL1:Q2.2, MOTOR_CONTROL1:Q3.2, MOTOR_CONTROL1:Q4.2, MOTOR_CONTROL1:R2.1, MOTOR_CONTROL1:R4.1, MOTOR_CONTROL1:R6.1, MOTOR_CONTROL1:R8.1
- net I2C_SCL: now also 03_MICROCONTROLLER:TP_SCL.TP, 03_MICROCONTROLLER:U301.29; no longer MICROCONTROLLER1:TP2.TP, MICROCONTROLLER1:U101.29
- net I2C_SDA: now also 03_MICROCONTROLLER:TP_SDA.TP, 03_MICROCONTROLLER:U301.30; no longer MICROCONTROLLER1:TP3.TP, MICROCONTROLLER1:U101.30
- net M1: now also 06_MOTOR_CONTROL:D601.A, 06_MOTOR_CONTROL:Q601.3; no longer MOTOR_CONTROL1:Q1.3, MOTOR_CONTROL1:U$1.P$1
- net M1_PWM: now also 03_MICROCONTROLLER:U301.18, 06_MOTOR_CONTROL:R601.1; no longer MICROCONTROLLER1:U101.18, MOTOR_CONTROL1:R1.1
- net M2: now also 06_MOTOR_CONTROL:D602.A, 06_MOTOR_CONTROL:Q602.3; no longer MOTOR_CONTROL1:Q2.3, MOTOR_CONTROL1:U$2.P$1
- net M2_PWM: now also 03_MICROCONTROLLER:U301.19, 06_MOTOR_CONTROL:R603.1; no longer MICROCONTROLLER1:U101.19, MOTOR_CONTROL1:R3.1
- net M3: now also 06_MOTOR_CONTROL:D603.A, 06_MOTOR_CONTROL:Q603.3; no longer MOTOR_CONTROL1:Q3.3, MOTOR_CONTROL1:U$3.P$1
- net M3_PWM: now also 03_MICROCONTROLLER:U301.20, 06_MOTOR_CONTROL:R605.1; no longer MICROCONTROLLER1:U101.20, MOTOR_CONTROL1:R5.1
- net M4: now also 06_MOTOR_CONTROL:D604.A, 06_MOTOR_CONTROL:Q604.3; no longer MOTOR_CONTROL1:Q4.3, MOTOR_CONTROL1:U$4.P$1
- net M4_PWM: now also 03_MICROCONTROLLER:U301.21, 06_MOTOR_CONTROL:R607.1; no longer MICROCONTROLLER1:U101.21, MOTOR_CONTROL1:R7.1
- net NRST: now also 03_MICROCONTROLLER:R301.2, 03_MICROCONTROLLER:U301.4, 07_CONNECTORS:X706.5; no longer CONNECTORS1:X6.5, MICROCONTROLLER1:R101.2, MICROCONTROLLER1:U101.4
- net SWCLK: now also 03_MICROCONTROLLER:U301.24, 07_CONNECTORS:X706.2; no longer CONNECTORS1:X6.2, MICROCONTROLLER1:U101.24
- net SWDIO: now also 03_MICROCONTROLLER:U301.23, 07_CONNECTORS:X706.4; no longer CONNECTORS1:X6.4, MICROCONTROLLER1:U101.23
- net UART1_RX: now also 03_MICROCONTROLLER:U301.9, 04_WIFI:U401.16; no longer MICROCONTROLLER1:U101.9, WIFI1:U301.16
- net UART1_TX: now also 03_MICROCONTROLLER:U301.8, 04_WIFI:U401.15; no longer MICROCONTROLLER1:U101.8, WIFI1:U301.15
Routing:
- added copper zone on layer 15, net GND
