File: Electronics/02_Board_files/01_Project files/V1_Flight_Controller/V1_Flight_Controller.sch (EAGLE design)
At the start: 27 parts, among them J101 JTAG_CONNECTOR, U101 STM32F030K6T6, U201 MPU-6050, Y1 8MHz

Commit message: 1. Created hierarchical structure in schematic 2. Battery charging and protection circuit added 3. Added various eagle libraries
Parts:
- removed C101, C102, C103, C104, C105, C106, C107: (no value), adafruit:C-USC0603
- removed C201: 0.1uF, 4V, ±10%, adafruit:C-USC0603
- removed C202: 10nF, 4V, ±10%, adafruit:C-USC0603
- removed C203: 2.2nF, 50V, ±10%, adafruit:C-USC0603
- removed C204: 0.1uF, 2V, ±10%, adafruit:C-USC0603
- removed J101: JTAG_CONNECTOR, con-molex:53047-05
- removed L101, L102, L103, L104, L201: (no value), rcl:L-USL2012C
- removed R101: (no value), adafruit:R-US_R0603
- removed R201, R202: 4.7k, adafruit:R-US_R0603
- removed TP1, TP2, TP3: TPB1,27, testpad:TPB1,27
- removed U101: STM32F030K6T6, STM32F030K6T6:STM32F030K6T6
- removed U201: MPU-6050, MPU-6050:MPU-6050
- removed U301: (no value), esp12e:ESP8266-12EESP12E
- removed Y1: 8MHz, SparkFun-Clocks:CRYSTAL-8MHZSMD-HC49UP
Connections:
- removed net 3V3: L101.2, L201.2, U301.VCC
- removed net 3V3_IMU: C201.1, C202.1, L201.1, R201.1, R202.1, U201.VDD, U201.VLOGIC
- removed net 3V3_MCU: C101.1, C102.1, C103.1, J101-1.S, L101.1, L102.2, L104.1, R101.1, TP1.TP, U101.VDD
- removed net BOOT0: L102.1, L103.1, U101.BOOT0
- removed net GND: U301.GND
- removed net GND_IMU: C201.2, C202.2, C203.2, C204.2, U201.AD0, U201.CLKIN, U201.FSYNC, U201.GND
- removed net GND_MCU: C101.2, C102.2, C103.2, C104.2, C105.2, C106.2, C107.2, J101-3.S, L103.2, U101.VSS
- removed net I2C1_SCL: TP2.TP, U101.PB6
- removed net I2C1_SDA: TP3.TP, U101.PB7
- removed net IMU_INT: U201.INT
- removed net N$1: C204.1, U201.REGOUT
- removed net N$2: C203.1, U201.CPOUT
- removed net NRST: J101-5.S, R101.2, U101.NRST
- removed net PWM_PIN1: U101.PA8
- removed net PWM_PIN2: U101.PA9
- removed net PWM_PIN3: U101.PA10
- removed net PWM_PIN4: U101.PA11
- removed net RST: U301.REST
- removed net SCL: R201.2, U201.SCL
- removed net SDA: R202.2, U201.SDA
- removed net SWCLK: J101-2.S, U101.PA14/SWCLK
- removed net SWDIO: J101-4.S, U101.PA13/SWDIO
- removed net USART1_RX: U101.PA3
- removed net USART1_TX: U101.PA2
- removed net VBAT_LEVEL: U101.PA0
- removed net VDDA: C104.1, C105.1, L104.2, U101.VDDA
- removed net XTAL_IN: C106.1, U101.PFO-OSC_IN/I2C1_SDA, Y1.1
- removed net XTAL_OUT: C107.1, U101.PF1-OSC_OUT/I2C1_SCL, Y1.2
